Commit message: Update for slow start
Signed-off-by: Wonho Yun <ywh@robotis.com>

File: ffw_description/ros2_control/ffw_bg2_rev4_follower/ffw_bg2_follower.ros2_control.xacro (robot description, xacro)
@@ -20,28 +20,48 @@
             <param name="baud_rate">4000000</param>
             <param name="dynamixel_model_folder">/param/dxl_model</param>
-            <param name="number_of_joints">9</param>
-            <param name="number_of_transmissions">9</param>
+            <param name="number_of_joints">19</param>
+            <param name="number_of_transmissions">19</param>
             <param name="disable_torque_at_init">true</param>
             <param name="transmission_to_joint_matrix">
-              1, 0, 0, 0, 0, 0, 0, 0, 0,
-              0, 1, 0, 0, 0, 0, 0, 0, 0,
-              0, 0, 1, 0, 0, 0, 0, 0, 0,
-              0, 0, 0, 1, 0, 0, 0, 0, 0,
-              0, 0, 0, 0, 1, 0, 0, 0, 0,
-              0, 0, 0, 0, 0, 1, 0, 0, 0,
-              0, 0, 0, 0, 0, 0, 1, 0, 0,
-              0, 0, 0, 0, 0, 0, 0, 1, 0,
-              0, 0, 0, 0, 0, 0, 0, 0, 1
+              1, 0, 0, 0, 0, 0, 0, 0, 0, 0, 0, 0, 0, 0, 0, 0, 0, 0, 0,
+              0, 1, 0, 0, 0, 0, 0, 0, 0, 0, 0, 0, 0, 0, 0, 0, 0, 0, 0,
+              0, 0, 1, 0, 0, 0, 0, 0, 0, 0, 0, 0, 0, 0, 0, 0, 0, 0, 0,
+              0, 0, 0, 1, 0, 0, 0, 0, 0, 0, 0, 0, 0, 0, 0, 0, 0, 0, 0,
+              0, 0, 0, 0, 1, 0, 0, 0, 0, 0, 0, 0, 0, 0, 0, 0, 0, 0, 0,
+              0, 0, 0, 0, 0, 1, 0, 0, 0, 0, 0, 0, 0, 0, 0, 0, 0, 0, 0,
+              0, 0, 0, 0, 0, 0, 1, 0, 0, 0, 0, 0, 0, 0, 0, 0, 0, 0, 0,
+              0, 0, 0, 0, 0, 0, 0, 1, 0, 0, 0, 0, 0, 0, 0, 0, 0, 0, 0,
+              0, 0, 0, 0, 0, 0, 0, 0, 1, 0, 0, 0, 0, 0, 0, 0, 0, 0, 0,
+              0, 0, 0, 0, 0, 0, 0, 0, 0, 1, 0, 0, 0, 0, 0, 0, 0, 0, 0,
+              0, 0, 0, 0, 0, 0, 0, 0, 0, 0, 1, 0, 0, 0, 0, 0, 0, 0, 0,
+              0, 0, 0, 0, 0, 0, 0, 0, 0, 0, 0, 1, 0, 0, 0, 0, 0, 0, 0,
+              0, 0, 0, 0, 0, 0, 0, 0, 0, 0, 0, 0, 1, 0, 0, 0, 0, 0, 0,
+              0, 0, 0, 0, 0, 0, 0, 0, 0, 0, 0, 0, 0, 1, 0, 0, 0, 0, 0,
+              0, 0, 0, 0, 0, 0, 0, 0, 0, 0, 0, 0, 0, 0, 1, 0, 0, 0, 0,
+              0, 0, 0, 0, 0, 0, 0, 0, 0, 0, 0, 0, 0, 0, 0, 1, 0, 0, 0,
+              0, 0, 0, 0, 0, 0, 0, 0, 0, 0, 0, 0, 0, 0, 0, 0, 1, 0, 0,
+              0, 0, 0, 0, 0, 0, 0, 0, 0, 0, 0, 0, 0, 0, 0, 0, 0, 1, 0,
+              0, 0, 0, 0, 0, 0, 0, 0, 0, 0, 0, 0, 0, 0, 0, 0, 0, 0, 1
             </param>
             <param name="joint_to_transmission_matrix">
-              1, 0, 0, 0, 0, 0, 0, 0, 0,
-              0, 1, 0, 0, 0, 0, 0, 0, 0,
-              0, 0, 1, 0, 0, 0, 0, 0, 0,
-              0, 0, 0, 1, 0, 0, 0, 0, 0,
-              0, 0, 0, 0, 1, 0, 0, 0, 0,
-              0, 0, 0, 0, 0, 1, 0, 0, 0,
-              0, 0, 0, 0, 0, 0, 1, 0, 0,
-              0, 0, 0, 0, 0, 0, 0, 1, 0,
-              0, 0, 0, 0, 0, 0, 0, 0, 1
+              1, 0, 0, 0, 0, 0, 0, 0, 0, 0, 0, 0, 0, 0, 0, 0, 0, 0, 0,
+              0, 1, 0, 0, 0, 0, 0, 0, 0, 0, 0, 0, 0, 0, 0, 0, 0, 0, 0,
+              0, 0, 1, 0, 0, 0, 0, 0, 0, 0, 0, 0, 0, 0, 0, 0, 0, 0, 0,
+              0, 0, 0, 1, 0, 0, 0, 0, 0, 0, 0, 0, 0, 0, 0, 0, 0, 0, 0,
+              0, 0, 0, 0, 1, 0, 0, 0, 0, 0, 0, 0, 0, 0, 0, 0, 0, 0, 0,
+              0, 0, 0, 0, 0, 1, 0, 0, 0, 0, 0, 0, 0, 0, 0, 0, 0, 0, 0,
+              0, 0, 0, 0, 0, 0, 1, 0, 0, 0, 0, 0, 0, 0, 0, 0, 0, 0, 0,
+              0, 0, 0, 0, 0, 0, 0, 1, 0, 0, 0, 0, 0, 0, 0, 0, 0, 0, 0,
+              0, 0, 0, 0, 0, 0, 0, 0, 1, 0, 0, 0, 0, 0, 0, 0, 0, 0, 0,
+              0, 0, 0, 0, 0, 0, 0, 0, 0, 1, 0, 0, 0, 0, 0, 0, 0, 0, 0,
+              0, 0, 0, 0, 0, 0, 0, 0, 0, 0, 1, 0, 0, 0, 0, 0, 0, 0, 0,
+              0, 0, 0, 0, 0, 0, 0, 0, 0, 0, 0, 1, 0, 0, 0, 0, 0, 0, 0,
+              0, 0, 0, 0, 0, 0, 0, 0, 0, 0, 0, 0, 1, 0, 0, 0, 0, 0, 0,
+              0, 0, 0, 0, 0, 0, 0, 0, 0, 0, 0, 0, 0, 1, 0, 0, 0, 0, 0,
+              0, 0, 0, 0, 0, 0, 0, 0, 0, 0, 0, 0, 0, 0, 1, 0, 0, 0, 0,
+              0, 0, 0, 0, 0, 0, 0, 0, 0, 0, 0, 0, 0, 0, 0, 1, 0, 0, 0,
+              0, 0, 0, 0, 0, 0, 0, 0, 0, 0, 0, 0, 0, 0, 0, 0, 1, 0, 0,
+              0, 0, 0, 0, 0, 0, 0, 0, 0, 0, 0, 0, 0, 0, 0, 0, 0, 1, 0,
+              0, 0, 0, 0, 0, 0, 0, 0, 0, 0, 0, 0, 0, 0, 0, 0, 0, 0, 1
             </param>
             <param name="dynamixel_state_pub_msg_name">dynamixel_hardware_interface/dxl_state</param>
@@ -50,5 +70,4 @@
             <param name="reboot_dxl_srv_name">dynamixel_hardware_interface/reboot_dxl</param>
             <param name="set_dxl_torque_srv_name">dynamixel_hardware_interface/set_dxl_torque</param>
-            <param name="error_timeout_ms">500</param>
           </xacro:unless>
         </hardware>
@@ -96,4 +115,64 @@
         <state_interface name="effort"/>
       </joint>
+      <joint name="gripper_r_joint1">
+        <command_interface name="position"/>
+        <state_interface name="position"/>
+        <state_interface name="velocity"/>
+        <state_interface name="effort"/>
+      </joint>
+      <joint name="arm_l_joint1">
+        <command_interface name="position"/>
+        <state_interface name="position"/>
+        <state_interface name="velocity"/>
+        <state_interface name="effort"/>
+      </joint>
+      <joint name="arm_l_joint2">
+        <command_interface name="position"/>
+        <state_interface name="position"/>
+        <state_interface name="velocity"/>
+        <state_interface name="effort"/>
+      </joint>
+      <joint name="arm_l_joint3">
+        <command_interface name="position"/>
+        <state_interface name="position"/>
+        <state_interface name="velocity"/>
+        <state_interface name="effort"/>
+      </joint>
+      <joint name="arm_l_joint4">
+        <command_interface name="position"/>
+        <state_interface name="position"/>
+        <state_interface name="velocity"/>
+        <state_interface name="effort"/>
+      </joint>
+      <joint name="arm_l_joint5">
+        <command_interface name="position"/>
+        <state_interface name="position"/>
+        <state_interface name="velocity"/>
+        <state_interface name="effort"/>
+      </joint>
+      <joint name="arm_l_joint6">
+        <command_interface name="position"/>
+        <state_interface name="position"/>
+        <state_interface name="velocity"/>
+        <state_interface name="effort"/>
+      </joint>
+      <joint name="arm_l_joint7">
+        <command_interface name="position"/>
+        <state_interface name="position"/>
+        <state_interface name="velocity"/>
+        <state_interface name="effort"/>
+      </joint>
+      <joint name="gripper_l_joint1">
+        <command_interface name="position"/>
+        <state_interface name="position"/>
+        <state_interface name="velocity"/>
+        <state_interface name="effort"/>
+      </joint>
+      <joint name="lift_joint">
+        <command_interface name="position"/>
+        <state_interface name="position"/>
+        <state_interface name="velocity"/>
+        <state_interface name="effort"/>
+      </joint>
       <joint name="head_joint1">
         <command_interface name="position"/>
@@ -117,13 +196,13 @@
         <state_interface name="Present Current"/>
         <state_interface name="Error Code"/>
-        <param name="Drive Mode">65</param>
+        <param name="Drive Mode">69</param>
         <param name="Operating Mode">3</param>
         <param name="Return Delay Time">0</param>
         <param name="Velocity Limit">3591</param>
         <param name="Acceleration Limit">35910</param>
-        <param name="Profile Velocity">359</param>
-        <param name="Profile Acceleration">359</param>
-        <!-- <param name="Profile Acceleration Time">750</param>
-        <param name="Profile Time">1500</param> -->
+        <param name="Profile Velocity">3591</param>
+        <param name="Profile Acceleration">3591</param>
+        <param name="Profile Acceleration Time">250</param>
+        <param name="Profile Time">500</param>
         <param name="Max Position Limit">262144</param>
         <param name="Min Position Limit">-262144</param>
@@ -141,13 +220,13 @@
         <state_interface name="Present Current"/>
         <state_interface name="Error Code"/>
-        <param name="Drive Mode">64</param>
+        <param name="Drive Mode">68</param>
         <param name="Operating Mode">3</param>
         <param name="Return Delay Time">0</param>
         <param name="Velocity Limit">3591</param>
         <param name="Acceleration Limit">35910</param>
-        <param name="Profile Velocity">359</param>
-        <param name="Profile Acceleration">359</param>
-        <!-- <param name="Profile Acceleration Time">750</param>
-        <param name="Profile Time">1500</param> -->
+        <param name="Profile Velocity">3591</param>
+        <param name="Profile Acceleration">3591</param>
+        <param name="Profile Acceleration Time">250</param>
+        <param name="Profile Time">500</param>
         <param name="Max Position Limit">0</param>
         <param name="Min Position Limit">-262144</param>
@@ -165,13 +244,13 @@
         <state_interface name="Present Current"/>
         <state_interface name="Error Code"/>
-        <param name="Drive Mode">65</param>
+        <param name="Drive Mode">69</param>
         <param name="Operating Mode">3</param>
         <param name="Return Delay Time">0</param>
         <param name="Velocity Limit">3591</param>
         <param name="Acceleration Limit">35910</param>
-        <param name="Profile Velocity">359</param>
-        <param name="Profile Acceleration">359</param>
-        <!-- <param name="Profile Acceleration Time">750</param>
-        <param name="Profile Time">1500</param> -->
+        <param name="Profile Velocity">3591</param>
+        <param name="Profile Acceleration">3591</param>
+        <param name="Profile Acceleration Time">250</param>
+        <param name="Profile Time">500</param>
         <param name="Max Position Limit">262144</param>
         <param name="Min Position Limit">-262144</param>
@@ -189,13 +268,13 @@
         <state_interface name="Present Current"/>
         <state_interface name="Error Code"/>
-        <param name="Drive Mode">65</param>
+        <param name="Drive Mode">69</param>
         <param name="Operating Mode">3</param>
         <param name="Return Delay Time">0</param>
         <param name="Velocity Limit">6486</param>
         <param name="Acceleration Limit">35910</param>
-        <param name="Profile Velocity">648</param>
-        <param name="Profile Acceleration">359</param>
-        <!-- <param name="Profile Acceleration Time">750</param>
-        <param name="Profile Time">1500</param> -->
+        <param name="Profile Velocity">6486</param>
+        <param name="Profile Acceleration">3591</param>
+        <param name="Profile Acceleration Time">250</param>
+        <param name="Profile Time">500</param>
         <param name="Max Position Limit">90000</param>
         <param name="Min Position Limit">-245000</param>
@@ -213,13 +292,13 @@
         <state_interface name="Present Current"/>
         <state_interface name="Error Code"/>
-        <param name="Drive Mode">65</param>
+        <param name="Drive Mode">69</param>
         <param name="Operating Mode">3</param>
         <param name="Return Delay Time">0</param>
         <param name="Velocity Limit">6486</param>
         <param name="Acceleration Limit">35910</param>
-        <param name="Profile Velocity">648</param>
-        <param name="Profile Acceleration">359</param>
-        <!-- <param name="Profile Acceleration Time">750</param>
-        <param name="Profile Time">1500</param> -->
+        <param name="Profile Velocity">6486</param>
+        <param name="Profile Acceleration">3591</param>
+        <param name="Profile Acceleration Time">250</param>
+        <param name="Profile Time">500</param>
         <param name="Max Position Limit">262144</param>
         <param name="Min Position Limit">-262144</param>
@@ -237,13 +316,13 @@
         <state_interface name="Present Current"/>
         <state_interface name="Error Code"/>
-        <param name="Drive Mode">65</param>
+        <param name="Drive Mode">69</param>
         <param name="Operating Mode">3</param>
         <param name="Return Delay Time">0</param>
         <param name="Velocity Limit">6486</param>
         <param name="Acceleration Limit">35910</param>
-        <param name="Profile Velocity">648</param>
-        <param name="Profile Acceleration">359</param>
-        <!-- <param name="Profile Acceleration Time">750</param>
-        <param name="Profile Time">1500</param> -->
+        <param name="Profile Velocity">6486</param>
+        <param name="Profile Acceleration">3591</param>
+        <param name="Profile Acceleration Time">250</param>
+        <param name="Profile Time">500</param>
         <param name="Max Position Limit">131072</param>
         <param name="Min Position Limit">-131072</param>
@@ -267,13 +346,227 @@
         <param name="Acceleration Limit">359100</param>
         <param name="Current Limit">1500</param>
-        <param name="Profile Velocity">300</param>
-        <param name="Profile Acceleration">150</param>
+        <param name="Profile Velocity">100</param>
+        <param name="Profile Acceleration">50</param>
         <param name="Max Position Limit">131875</param>
         <param name="Min Position Limit">-151875</param>
       </gpio>
+      <gpio name="dxl8">
+        <param name="type">dxl</param>
+        <param name="ID">8</param>
+        <command_interface name="Goal Position"/>
+        <state_interface name="Present Position"/>
+        <state_interface name="Present Velocity"/>
+        <state_interface name="Present Current"/>
+        <state_interface name="Hardware Error Status"/>
+        <param name="Operating Mode">5</param>
+        <param name="Return Delay Time">0</param>
+        <param name="Profile Velocity">0</param>
+        <param name="Profile Acceleration">0</param>
+      </gpio>
+      <!-- LEFT ARM -->
+      <gpio name="dxl31">
+        <param name="type">dxl</param>
+        <param name="ID">31</param>
+        <command_interface name="Goal Position"/>
+        <state_interface name="Present Position"/>
+        <state_interface name="Present Velocity"/>
+        <state_interface name="Present Current"/>
+        <state_interface name="Error Code"/>
+        <param name="Drive Mode">68</param>
+        <param name="Operating Mode">3</param>
+        <param name="Return Delay Time">0</param>
+        <param name="Velocity Limit">3591</param>
+        <param name="Acceleration Limit">35910</param>
+        <param name="Profile Velocity">3591</param>
+        <param name="Profile Acceleration">3591</param>
+        <param name="Profile Acceleration Time">250</param>
+        <param name="Profile Time">500</param>
+        <param name="Max Position Limit">262144</param>
+        <param name="Min Position Limit">-262144</param>
+        <param name="Position P Gain">1583185</param>
+        <param name="Velocity P Gain">41387</param>
+        <param name="Velocity I Gain">1565630</param>
+        <param name="Position FF Gain">100</param>
+      </gpio>
+      <gpio name="dxl32">
+        <param name="type">dxl</param>
+        <param name="ID">32</param>
+        <command_interface name="Goal Position"/>
+        <state_interface name="Present Position"/>
+        <state_interface name="Present Velocity"/>
+        <state_interface name="Present Current"/>
+        <state_interface name="Error Code"/>
+        <param name="Drive Mode">68</param>
+        <param name="Operating Mode">3</param>
+        <param name="Return Delay Time">0</param>
+        <param name="Velocity Limit">3591</param>
+        <param name="Acceleration Limit">35910</param>
+        <param name="Profile Velocity">3591</param>
+        <param name="Profile Acceleration">3591</param>
+        <param name="Profile Acceleration Time">250</param>
+        <param name="Profile Time">500</param>
+        <param name="Max Position Limit">262144</param>
+        <param name="Min Position Limit">0</param>
+        <param name="Position P Gain">1583185</param>
+        <param name="Velocity P Gain">41387</param>
+        <param name="Velocity I Gain">1565630</param>
+        <param name="Position FF Gain">100</param>
+      </gpio>
+      <gpio name="dxl33">
+        <param name="type">dxl</param>
+        <param name="ID">33</param>
+        <command_interface name="Goal Position"/>
+        <state_interface name="Present Position"/>
+        <state_interface name="Present Velocity"/>
+        <state_interface name="Present Current"/>
+        <state_interface name="Error Code"/>
+        <param name="Drive Mode">69</param>
+        <param name="Operating Mode">3</param>
+        <param name="Return Delay Time">0</param>
+        <param name="Velocity Limit">3591</param>
+        <param name="Acceleration Limit">35910</param>
+        <param name="Profile Velocity">3591</param>
+        <param name="Profile Acceleration">3591</param>
+        <param name="Profile Acceleration Time">250</param>
+        <param name="Profile Time">500</param>
+        <param name="Max Position Limit">262144</param>
+        <param name="Min Position Limit">-262144</param>
+        <param name="Position P Gain">1583185</param>
+        <param name="Velocity P Gain">41387</param>
+        <param name="Velocity I Gain">1565630</param>
+        <param name="Position FF Gain">100</param>
+      </gpio>
+      <gpio name="dxl34">
+        <param name="type">dxl</param>
+        <param name="ID">34</param>
+        <command_interface name="Goal Position"/>
+        <state_interface name="Present Position"/>
+        <state_interface name="Present Velocity"/>
+        <state_interface name="Present Current"/>
+        <state_interface name="Error Code"/>
+        <param name="Drive Mode">68</param>
+        <param name="Operating Mode">3</param>
+        <param name="Return Delay Time">0</param>
+        <param name="Velocity Limit">6486</param>
+        <param name="Acceleration Limit">35910</param>
+        <param name="Profile Velocity">6486</param>
+        <param name="Profile Acceleration">3591</param>
+        <param name="Profile Acceleration Time">250</param>
+        <param name="Profile Time">500</param>
+        <param name="Max Position Limit">90000</param>
+        <param name="Min Position Limit">-245000</param>
+        <param name="Position P Gain">1583185</param>
+        <param name="Velocity P Gain">18184</param>
+        <param name="Velocity I Gain">1585331</param>
+        <param name="Position FF Gain">100</param>
+      </gpio>
+      <gpio name="dxl35">
+        <param name="type">dxl</param>
+        <param name="ID">35</param>
+        <command_interface name="Goal Position"/>
+        <state_interface name="Present Position"/>
+        <state_interface name="Present Velocity"/>
+        <state_interface name="Present Current"/>
+        <state_interface name="Error Code"/>
+        <param name="Drive Mode">69</param>
+        <param name="Operating Mode">3</param>
+        <param name="Return Delay Time">0</param>
+        <param name="Velocity Limit">6486</param>
+        <param name="Acceleration Limit">35910</param>
+        <param name="Profile Velocity">6486</param>
+        <param name="Profile Acceleration">3591</param>
+        <param name="Profile Acceleration Time">250</param>
+        <param name="Profile Time">500</param>
+        <param name="Max Position Limit">262144</param>
+        <param name="Min Position Limit">-262144</param>
+        <param name="Position P Gain">1583185</param>
+        <param name="Velocity P Gain">18184</param>
+        <param name="Velocity I Gain">1585331</param>
+        <param name="Position FF Gain">100</param>
+      </gpio>
+      <gpio name="dxl36">
+        <param name="type">dxl</param>
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
File: ffw_description/urdf/common/follower/ffw_follower_body.xacro (robot description, xacro)
@@ -13,5 +13,5 @@
          <dynamics damping="0.1" />
       </joint>
-      <!-- <joint name="${prefix}lift_joint" type="fixed">
+      <joint name="${prefix}lift_joint" type="fixed">
          <parent link="${parent}"/>
          <child link="${prefix}arm_base_link" />
@@ -20,5 +20,5 @@
          <limit velocity="4.8" effort="1000" lower="-0.5" upper="0.0" />
          <dynamics damping="0.1" />
-      </joint> -->
+      </joint>
       <link name="${prefix}arm_base_link">
          <visual>

File: ffw_description/urdf/ffw_bg2_rev4_follower/ffw_bg2_follower.urdf.xacro (robot description, xacro)
@@ -10,5 +10,4 @@
   <xacro:include filename="$(find ffw_description)/urdf/common/rh_p12_rn_a/rh_p12_rn_a.urdf.xacro" />
   <xacro:include filename="$(find ffw_description)/ros2_control/$(arg model)/ffw_bg2_follower.ros2_control.xacro" />
-  <xacro:include filename="$(find ffw_description)/ros2_control/$(arg model)/ffw_bg2_follower_left.ros2_control.xacro" />
   <xacro:include filename="$(find ffw_description)/gazebo/$(arg model)/ffw_bg2_follower.gazebo.xacro" />
   <link name="world"/>
@@ -87,8 +86,4 @@
     use_fake_hardware="$(arg use_fake_hardware)"
     fake_sensor_commands="$(arg fake_sensor_commands)"/>
-  <xacro:ffw_bg2_follower_left_system
-    use_sim="$(arg use_sim)"
-    use_fake_hardware="$(arg use_fake_hardware)"
-    fake_sensor_commands="$(arg fake_sensor_commands)"/>
   <gazebo>
       <plugin filename="gz_ros2_control-system" name="gz_ros2_control::GazeboSimROS2ControlPlugin">
