Commit message: Add support for bh5 gz
Signed-off-by: Wonho Yun <ywh@robotis.com>

File: ffw_description/ros2_control/ffw_bh5_rev1_follower/ffw_bh5_follower.ros2_control.xacro (robot description, xacro)
@@ -191,10 +191,10 @@
         <state_interface name="effort"/>
       </joint>
-      <joint name="gripper_r_joint1">
-        <command_interface name="position"/>
-        <state_interface name="position"/>
-        <state_interface name="velocity"/>
-        <state_interface name="effort"/>
-      </joint>
+      <!-- <joint name="gripper_r_joint1">
+        <command_interface name="position"/>
+        <state_interface name="position"/>
+        <state_interface name="velocity"/>
+        <state_interface name="effort"/>
+      </joint> -->
       <joint name="arm_l_joint1">
         <command_interface name="position"/>
@@ -239,10 +239,10 @@
         <state_interface name="effort"/>
       </joint>
-      <joint name="gripper_l_joint1">
-        <command_interface name="position"/>
-        <state_interface name="position"/>
-        <state_interface name="velocity"/>
-        <state_interface name="effort"/>
-      </joint>
+      <!-- <joint name="gripper_l_joint1">
+        <command_interface name="position"/>
+        <state_interface name="position"/>
+        <state_interface name="velocity"/>
+        <state_interface name="effort"/>
+      </joint> -->
       <joint name="lift_joint">
         <command_interface name="position"/>
@@ -263,425 +263,4 @@
         <state_interface name="effort"/>
       </joint>
-      <!-- RIGHT ARM -->
-      <gpio name="dxl1">
-        <param name="type">dxl</param>
-        <param name="ID">1</param>
-        <command_interface name="Goal Position"/>
-        <state_interface name="Present Position"/>
-        <state_interface name="Present Velocity"/>
-        <state_interface name="Present Current"/>
-        <state_interface name="Error Code"/>
-        <param name="Drive Mode">69</param>
-        <param name="Operating Mode">3</param>
-        <param name="Return Delay Time">0</param>
-        <param name="Velocity Limit">3591</param>
-        <param name="Acceleration Limit">35910</param>
-        <param name="Profile Velocity">3591</param>
-        <param name="Profile Acceleration">3591</param>
-        <param name="Profile Acceleration Time">250</param>
-        <param name="Profile Time">500</param>
-        <param name="Max Position Limit">262144</param>
-        <param name="Min Position Limit">-262144</param>
-        <param name="Position P Gain">1583185</param>
-        <param name="Velocity P Gain">41387</param>
-        <param name="Velocity I Gain">1565630</param>
-        <param name="Position FF Gain">100</param>
-      </gpio>
-      <gpio name="dxl2">
-        <param name="type">dxl</param>
-        <param name="ID">2</param>
-        <command_interface name="Goal Position"/>
-        <state_interface name="Present Position"/>
-        <state_interface name="Present Velocity"/>
-        <state_interface name="Present Current"/>
-        <state_interface name="Error Code"/>
-        <param name="Drive Mode">68</param>
-        <param name="Operating Mode">3</param>
-        <param name="Return Delay Time">0</param>
-        <param name="Velocity Limit">3591</param>
-        <param name="Acceleration Limit">35910</param>
-        <param name="Profile Velocity">3591</param>
-        <param name="Profile Acceleration">3591</param>
-        <param name="Profile Acceleration Time">250</param>
-        <param name="Profile Time">500</param>
-        <param name="Max Position Limit">0</param>
-        <param name="Min Position Limit">-262144</param>
-        <param name="Position P Gain">1583185</param>
-        <param name="Velocity P Gain">41387</param>
-        <param name="Velocity I Gain">1565630</param>
-        <param name="Position FF Gain">100</param>
-      </gpio>
-      <gpio name="dxl3">
-        <param name="type">dxl</param>
-        <param name="ID">3</param>
-        <command_interface name="Goal Position"/>
-        <state_interface name="Present Position"/>
-        <state_interface name="Present Velocity"/>
-        <state_interface name="Present Current"/>
-        <state_interface name="Error Code"/>
-        <param name="Drive Mode">69</param>
-        <param name="Operating Mode">3</param>
-        <param name="Return Delay Time">0</param>
-        <param name="Velocity Limit">3591</param>
-        <param name="Acceleration Limit">35910</param>
-        <param name="Profile Velocity">3591</param>
-        <param name="Profile Acceleration">3591</param>
-        <param name="Profile Acceleration Time">250</param>
-        <param name="Profile Time">500</param>
-        <param name="Max Position Limit">262144</param>
-        <param name="Min Position Limit">-262144</param>
-        <param name="Position P Gain">1583185</param>
-        <param name="Velocity P Gain">41387</param>
-        <param name="Velocity I Gain">1565630</param>
-        <param name="Position FF Gain">100</param>
-      </gpio>
-      <gpio name="dxl4">
-        <param name="type">dxl</param>
-        <param name="ID">4</param>
-        <command_interface name="Goal Position"/>
-        <state_interface name="Present Position"/>
-        <state_interface name="Present Velocity"/>
-        <state_interface name="Present Current"/>
-        <state_interface name="Error Code"/>
-        <param name="Drive Mode">69</param>
-        <param name="Operating Mode">3</param>
-        <param name="Return Delay Time">0</param>
-        <param name="Velocity Limit">6486</param>
-        <param name="Acceleration Limit">35910</param>
-        <param name="Profile Velocity">6486</param>
-        <param name="Profile Acceleration">3591</param>
-        <param name="Profile Acceleration Time">250</param>
-        <param name="Profile Time">500</param>
-        <param name="Max Position Limit">90000</param>
-        <param name="Min Position Limit">-245000</param>
-        <param name="Position P Gain">1583185</param>
-        <param name="Velocity P Gain">18184</param>
-        <param name="Velocity I Gain">1585331</param>
-        <param name="Position FF Gain">100</param>
-      </gpio>
-      <gpio name="dxl5">
-        <param name="type">dxl</param>
-        <param name="ID">5</param>
-        <command_interface name="Goal Position"/>
-        <state_interface name="Present Position"/>
-        <state_interface name="Present Velocity"/>
-        <state_interface name="Present Current"/>
-        <state_interface name="Error Code"/>
-        <param name="Drive Mode">69</param>
-        <param name="Operating Mode">3</param>
-        <param name="Return Delay Time">0</param>
-        <param name="Velocity Limit">6486</param>
-        <param name="Acceleration Limit">35910</param>
-        <param name="Profile Velocity">6486</param>
-        <param name="Profile Acceleration">3591</param>
-        <param name="Profile Acceleration Time">250</param>
-        <param name="Profile Time">500</param>
-        <param name="Max Position Limit">262144</param>
-        <param name="Min Position Limit">-262144</param>
-        <param name="Position P Gain">1583185</param>
-        <param name="Velocity P Gain">18184</param>
-        <param name="Velocity I Gain">1585331</param>
-        <param name="Position FF Gain">100</param>
-      </gpio>
-      <gpio name="dxl6">
-        <param name="type">dxl</param>
-        <param name="ID">6</param>
-        <command_interface name="Goal Position"/>
-        <state_interface name="Present Position"/>
-        <state_interface name="Present Velocity"/>
-        <state_interface name="Present Current"/>
-        <state_interface name="Error Code"/>
-        <param name="Drive Mode">69</param>
-        <param name="Operating Mode">3</param>
-        <param name="Return Delay Time">0</param>
-        <param name="Velocity Limit">6486</param>
-        <param name="Acceleration Limit">35910</param>
-        <param name="Profile Velocity">6486</param>
-        <param name="Profile Acceleration">3591</param>
-        <param name="Profile Acceleration Time">250</param>
-        <param name="Profile Time">500</param>
-        <param name="Max Position Limit">131072</param>
-        <param name="Min Position Limit">-131072</param>
-        <param name="Position P Gain">1583185</param>
-        <param name="Velocity P Gain">18184</param>
-        <param name="Velocity I Gain">1585331</param>
-        <param name="Position FF Gain">100</param>
-      </gpio>
-      <gpio name="dxl7">
-        <param name="type">dxl</param>
-        <param name="ID">7</param>
-        <command_interface name="Goal Position"/>
-        <state_interface name="Present Position"/>
-        <state_interface name="Present Velocity"/>
-        <state_interface name="Present Current"/>
-        <state_interface name="Hardware Error Status"/>
-        <param name="Drive Mode">4</param>
-        <param name="Operating Mode">3</param>
-        <param name="Return Delay Time">0</param>
-        <param name="Velocity Limit">2920</param>
-        <param name="Acceleration Limit">359100</param>
-        <param name="Current Limit">1500</param>
-        <param name="Profile Velocity">100</param>
-        <param name="Profile Acceleration">50</param>
-        <param name="Max Position Limit">131875</param>
-        <param name="Min Position Limit">-151875</param>
-      </gpio>
-      <gpio name="dxl8">
-        <param name="type">dxl</param>
-        <param name="ID">8</param>
-        <command_interface name="Goal Position"/>
-        <state_interface name="Present Position"/>
-        <state_interface name="Present Velocity"/>
-        <state_interface name="Present Current"/>
-        <state_interface name="Hardware Error Status"/>
-        <param name="Operating Mode">5</param>
-        <param name="Return Delay Time">0</param>
-        <param name="Profile Velocity">0</param>
-        <param name="Profile Acceleration">0</param>
-      </gpio>
-      <!-- LEFT ARM -->
-      <gpio name="dxl31">
-        <param name="type">dxl</param>
-        <param name="ID">31</param>
-        <command_interface name="Goal Position"/>
-        <state_interface name="Present Position"/>
-        <state_interface name="Present Velocity"/>
-        <state_interface name="Present Current"/>
-        <state_interface name="Error Code"/>
-        <param name="Drive Mode">68</param>
-        <param name="Operating Mode">3</param>
-        <param name="Return Delay Time">0</param>
-        <param name="Velocity Limit">3591</param>
-        <param name="Acceleration Limit">35910</param>
-        <param name="Profile Velocity">3591</param>
-        <param name="Profile Acceleration">3591</param>
-        <param name="Profile Acceleration Time">250</param>
-        <param name="Profile Time">500</param>
-        <param name="Max Position Limit">262144</param>
-        <param name="Min Position Limit">-262144</param>
-        <param name="Position P Gain">1583185</param>
-        <param name="Velocity P Gain">41387</param>
-        <param name="Velocity I Gain">1565630</param>
-        <param name="Position FF Gain">100</param>
-      </gpio>
-      <gpio name="dxl32">
-        <param name="type">dxl</param>
-        <param name="ID">32</param>
-        <command_interface name="Goal Position"/>
-        <state_interface name="Present Position"/>
-        <state_interface name="Present Velocity"/>
-        <state_interface name="Present Current"/>
-        <state_interface name="Error Code"/>
-        <param name="Drive Mode">68</param>
-        <param name="Operating Mode">3</param>
-        <param name="Return Delay Time">0</param>
-        <param name="Velocity Limit">3591</param>
-        <param name="Acceleration Limit">35910</param>
-        <param name="Profile Velocity">3591</param>
-        <param name="Profile Acceleration">3591</param>
-        <param name="Profile Acceleration Time">250</param>
-        <param name="Profile Time">500</param>
-        <param name="Max Position Limit">262144</param>
-        <param name="Min Position Limit">0</param>
-        <param name="Position P Gain">1583185</param>
-        <param name="Velocity P Gain">41387</param>
-        <param name="Velocity I Gain">1565630</param>
-        <param name="Position FF Gain">100</param>
-      </gpio>
-      <gpio name="dxl33">
-        <param name="type">dxl</param>
-        <param name="ID">33</param>
-        <command_interface name="Goal Position"/>
-        <state_interface name="Present Position"/>
-        <state_interface name="Present Velocity"/>
-        <state_interface name="Present Current"/>
-        <state_interface name="Error Code"/>
-        <param name="Drive Mode">69</param>
-        <param name="Operating Mode">3</param>
-        <param name="Return Delay Time">0</param>
-        <param name="Velocity Limit">3591</param>
-        <param name="Acceleration Limit">35910</param>
-        <param name="Profile Velocity">3591</param>
-        <param name="Profile Acceleration">3591</param>
-        <param name="Profile Acceleration Time">250</param>
-        <param name="Profile Time">500</param>
-        <param name="Max Position Limit">262144</param>
-        <param name="Min Position Limit">-262144</param>
-        <param name="Position P Gain">1583185</param>
-        <param name="Velocity P Gain">41387</param>
-        <param name="Velocity I Gain">1565630</param>
-        <param name="Position FF Gain">100</param>
-      </gpio>
-      <gpio name="dxl34">
-        <param name="type">dxl</param>
-        <param name="ID">34</param>
-        <command_interface name="Goal Position"/>
-        <state_interface name="Present Position"/>
-        <state_interface name="Present Velocity"/>
-        <state_interface name="Present Current"/>
-        <state_interface name="Error Code"/>
-        <param name="Drive Mode">68</param>
-        <param name="Operating Mode">3</param>
-        <param name="Return Delay Time">0</param>
-        <param name="Velocity Limit">6486</param>
-        <param name="Acceleration Limit">35910</param>
-        <param name="Profile Velocity">6486</param>
-        <param name="Profile Acceleration">3591</param>
-        <param name="Profile Acceleration Time">250</param>
-        <param name="Profile Time">500</param>
-        <param name="Max Position Limit">90000</param>
-        <param name="Min Position Limit">-245000</param>
-        <param name="Position P Gain">1583185</param>
-        <param name="Velocity P Gain">18184</param>
-        <param name="Velocity I Gain">1585331</param>
-        <param name="Position FF Gain">100</param>
-      </gpio>
-      <gpio name="dxl35">
-        <param name="type">dxl</param>
-        <param name="ID">35</param>
-        <command_interface name="Goal Position"/>
-        <state_interface name="Present Position"/>
-        <state_interface name="Present Velocity"/>
-        <state_interface name="Present Current"/>
-        <state_interface name="Error Code"/>
-        <param name="Drive Mode">69</param>
-        <param name="Operating Mode">3</param>
-        <param name="Return Delay Time">0</param>
-        <param name="Velocity Limit">6486</param>
-        <param name="Acceleration Limit">35910</param>
-        <param name="Profile Velocity">6486</param>
-        <param name="Profile Acceleration">3591</param>
-        <param name="Profile Acceleration Time">250</param>
-        <param name="Profile Time">500</param>
-        <param name="Max Position Limit">262144</param>
-        <param name="Min Position Limit">-262144</param>
-        <param name="Position P Gain">1583185</param>
-        <param name="Velocity P Gain">18184</param>
-        <param name="Velocity I Gain">1585331</param>
-        <param name="Position FF Gain">100</param>
-      </gpio>
-      <gpio name="dxl36">
-        <param name="type">dxl</param>
-        <param name="ID">36</param>
-        <command_interface name="Goal Position"/>
-        <state_interface name="Present Position"/>
-        <state_interface name="Present Velocity"/>
-        <state_interface name="Present Current"/>
-        <state_interface name="Error Code"/>
-        <param name="Drive Mode">68</param>
-        <param name="Operating Mode">3</param>
-        <param name="Return Delay Time">0</param>
-        <param name="Velocity Limit">6486</param>
-        <param name="Acceleration Limit">35910</param>
-        <param name="Profile Velocity">6486</param>
-        <param name="Profile Acceleration">3591</param>
-        <param name="Profile Acceleration Time">250</param>
-        <param name="Profile Time">500</param>
-        <param name="Max Position Limit">131072</param>
-        <param name="Min Position Limit">-131072</param>
-        <param name="Position P Gain">1583185</param>
-        <param name="Velocity P Gain">18184</param>
-        <param name="Velocity I Gain">1585331</param>
-        <param name="Position FF Gain">100</param>
-      </gpio>
-      <gpio name="dxl37">
-        <param name="type">dxl</param>
-        <param name="ID">37</param>
-        <command_interface name="Goal Position"/>
-        <state_interface name="Present Position"/>
-        <state_interface name="Present Velocity"/>
-        <state_interface name="Present Current"/>
-        <state_interface name="Hardware Error Status"/>
-        <param name="Drive Mode">4</param>
-        <param name="Operating Mode">3</param>
-        <param name="Return Delay Time">0</param>
-        <param name="Velocity Limit">2920</param>
-        <param name="Acceleration Limit">359100</param>
-        <param name="Current Limit">1500</param>
-        <param name="Profile Velocity">100</param>
-        <param name="Profile Acceleration">50</param>
-        <param name="Max Position Limit">131875</param>
-        <param name="Min Position Limit">-151875</param>
-      </gpio>
-      <gpio name="dxl38">
-        <param name="type">dxl</param>
-        <param name="ID">38</param>
-        <command_interface name="Goal Position"/>
-        <state_interface name="Present Position"/>
-        <state_interface name="Present Velocity"/>
-        <state_interface name="Present Current"/>
-        <state_interface name="Hardware Error Status"/>
-        <param name="Operating Mode">5</param>
-        <param name="Return Delay Time">0</param>
-        <param name="Profile Velocity">0</param>
-        <param name="Profile Acceleration">0</param>
-      </gpio>
-      <!-- LIFT -->
-      <gpio name="dxl81">
-        <param name="type">dxl</param>
-        <param name="ID">81</param>
-        <command_interface name="Goal Position"/>
-        <state_interface name="Present Position"/>
-        <state_interface name="Present Velocity"/>
-        <state_interface name="Present Current"/>
-        <state_interface name="Error Code"/>
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
File: ffw_description/urdf/ffw_bh5_rev1_follower/ffw_bh5_follower.urdf.xacro (robot description, xacro)
@@ -12,5 +12,5 @@
   <xacro:include filename="$(find ffw_description)/urdf/common/rh_5_right/rh_5_right.urdf.xacro" />
   <xacro:include filename="$(find ffw_description)/ros2_control/$(arg model)/ffw_bh5_follower.ros2_control.xacro" />
-  <xacro:include filename="$(find ffw_description)/gazebo/ffw_bg2_rev4_follower/ffw_bg2_follower.gazebo.xacro" />
+  <xacro:include filename="$(find ffw_description)/gazebo/ffw_bh5_rev1_follower/ffw_bh5_follower.gazebo.xacro" />
   <link name="world"/>
   <joint name="$(arg prefix)world_fixed" type="fixed">
@@ -61,5 +61,5 @@
   <gazebo>
       <plugin filename="gz_ros2_control-system" name="gz_ros2_control::GazeboSimROS2ControlPlugin">
-        <parameters>$(find ffw_bringup)/config/$(arg model)/ffw_bg2_follower_ai_hardware_controller.yaml</parameters>
+        <parameters>$(find ffw_bringup)/config/$(arg model)/ffw_bh5_follower_ai_hardware_controller.yaml</parameters>
       </plugin>
   </gazebo>
