Commit message: rename hx5

File: ffw_description/urdf/common/hx5_d20_right/hx5_d20_right.urdf.xacro (robot description, xacro)
@@ -1,25 +1,25 @@
 <?xml version="1.0" encoding="UTF-8"?>
 <robot xmlns:xacro="http://www.ros.org/wiki/xacro">
-   <xacro:macro name="rh_5_right" params="prefix parent *origin">
-      <xacro:property name="meshes_file_direction" value="package://ffw_description/meshes/common/rh_5_right/" />
-      <joint name="${prefix}rh_5_right_joint" type="fixed">
+   <xacro:macro name="hx5_d20_right" params="prefix parent *origin">
+      <xacro:property name="meshes_file_direction" value="package://ffw_description/meshes/common/hx5_d20_right/" />
+      <joint name="${prefix}hx5_d20_right_joint" type="fixed">
          <xacro:insert_block name="origin" />
          <parent link="${parent}"/>
-         <child link="${prefix}rh_5_right_base" />
-      </joint>
-      <link name="${prefix}rh_5_right_base">
-         <visual>
-            <origin xyz="0 0 0" rpy="0 0 0" />
-            <geometry>
-               <mesh filename="${meshes_file_direction}/rh_5_base_unit.stl" scale="0.001 0.001 0.001" />
-            </geometry>
-            <material name="grey">
-               <color rgba="0.2 0.2 0.2 1" />
-            </material>
-         </visual>
-         <collision>
-            <origin xyz="0 0 0" rpy="0 0 0" />
-            <geometry>
-               <mesh filename="${meshes_file_direction}/rh_5_base_unit.stl" scale="0.001 0.001 0.001" />
+         <child link="${prefix}hx5_d20_right_base" />
+      </joint>
+      <link name="${prefix}hx5_d20_right_base">
+         <visual>
+            <origin xyz="0 0 0" rpy="0 0 0" />
+            <geometry>
+               <mesh filename="${meshes_file_direction}/hx5_d20_base_unit.stl" scale="0.001 0.001 0.001" />
+            </geometry>
+            <material name="grey">
+               <color rgba="0.2 0.2 0.2 1" />
+            </material>
+         </visual>
+         <collision>
+            <origin xyz="0 0 0" rpy="0 0 0" />
+            <geometry>
+               <mesh filename="${meshes_file_direction}/hx5_d20_base_unit.stl" scale="0.001 0.001 0.001" />
             </geometry>
             <material name="grey">
@@ -37,5 +37,5 @@
       <!-- THUMB -->
       <joint name="${prefix}finger_r_joint1" type="revolute">
-         <parent link="${prefix}rh_5_right_base" />
+         <parent link="${prefix}hx5_d20_right_base" />
          <child link="${prefix}finger_r_link1" />
          <origin xyz="0.0145 0.02624 0.05394" rpy="-0.523599 0 0" />
@@ -48,14 +48,14 @@
             <origin xyz="0 0 0" rpy="0 0 0" />
             <geometry>
-               <mesh filename="${meshes_file_direction}/rh_5_thumb_mcp.stl" scale="0.001 0.001 0.001" />
-            </geometry>
-            <material name="grey">
-               <color rgba="0.2 0.2 0.2 1" />
-            </material>
-         </visual>
-         <collision>
-            <origin xyz="0 0 0" rpy="0 0 0" />
-            <geometry>
-               <mesh filename="${meshes_file_direction}/rh_5_thumb_mcp.stl" scale="0.001 0.001 0.001" />
+               <mesh filename="${meshes_file_direction}/hx5_d20_thumb_mcp.stl" scale="0.001 0.001 0.001" />
+            </geometry>
+            <material name="grey">
+               <color rgba="0.2 0.2 0.2 1" />
+            </material>
+         </visual>
+         <collision>
+            <origin xyz="0 0 0" rpy="0 0 0" />
+            <geometry>
+               <mesh filename="${meshes_file_direction}/hx5_d20_thumb_mcp.stl" scale="0.001 0.001 0.001" />
             </geometry>
             <material name="grey">
@@ -83,14 +83,14 @@
             <origin xyz="0 0 0" rpy="0 0 0" />
             <geometry>
-               <mesh filename="${meshes_file_direction}/rh_5_thumb_mcp2.stl" scale="0.001 0.001 0.001" />
-            </geometry>
-            <material name="grey">
-               <color rgba="0.2 0.2 0.2 1" />
-            </material>
-         </visual>
-         <collision>
-            <origin xyz="0 0 0" rpy="0 0 0" />
-            <geometry>
-               <mesh filename="${meshes_file_direction}/rh_5_thumb_mcp2.stl" scale="0.001 0.001 0.001" />
+               <mesh filename="${meshes_file_direction}/hx5_d20_thumb_mcp2.stl" scale="0.001 0.001 0.001" />
+            </geometry>
+            <material name="grey">
+               <color rgba="0.2 0.2 0.2 1" />
+            </material>
+         </visual>
+         <collision>
+            <origin xyz="0 0 0" rpy="0 0 0" />
+            <geometry>
+               <mesh filename="${meshes_file_direction}/hx5_d20_thumb_mcp2.stl" scale="0.001 0.001 0.001" />
             </geometry>
             <material name="grey">
@@ -118,14 +118,14 @@
             <origin xyz="0 0 0" rpy="0 0 0" />
             <geometry>
-               <mesh filename="${meshes_file_direction}/rh_5_thumb_ip.stl" scale="0.001 0.001 0.001" />
-            </geometry>
-            <material name="grey">
-               <color rgba="0.2 0.2 0.2 1" />
-            </material>
-         </visual>
-         <collision>
-            <origin xyz="0 0 0" rpy="0 0 0" />
-            <geometry>
-               <mesh filename="${meshes_file_direction}/rh_5_thumb_ip.stl" scale="0.001 0.001 0.001" />
+               <mesh filename="${meshes_file_direction}/hx5_d20_thumb_ip.stl" scale="0.001 0.001 0.001" />
+            </geometry>
+            <material name="grey">
+               <color rgba="0.2 0.2 0.2 1" />
+            </material>
+         </visual>
+         <collision>
+            <origin xyz="0 0 0" rpy="0 0 0" />
+            <geometry>
+               <mesh filename="${meshes_file_direction}/hx5_d20_thumb_ip.stl" scale="0.001 0.001 0.001" />
             </geometry>
             <material name="grey">
@@ -153,14 +153,14 @@
             <origin xyz="0 0 0" rpy="0 0 0" />
             <geometry>
-               <mesh filename="${meshes_file_direction}/rh_5_thumb_tip.stl" scale="0.001 0.001 0.001" />
-            </geometry>
-            <material name="grey">
-               <color rgba="0.2 0.2 0.2 1" />
-            </material>
-         </visual>
-         <collision>
-            <origin xyz="0 0 0" rpy="0 0 0" />
-            <geometry>
-               <mesh filename="${meshes_file_direction}/rh_5_thumb_tip.stl" scale="0.001 0.001 0.001" />
+               <mesh filename="${meshes_file_direction}/hx5_d20_thumb_tip.stl" scale="0.001 0.001 0.001" />
+            </geometry>
+            <material name="grey">
+               <color rgba="0.2 0.2 0.2 1" />
+            </material>
+         </visual>
+         <collision>
+            <origin xyz="0 0 0" rpy="0 0 0" />
+            <geometry>
+               <mesh filename="${meshes_file_direction}/hx5_d20_thumb_tip.stl" scale="0.001 0.001 0.001" />
             </geometry>
             <material name="grey">
@@ -194,5 +194,5 @@
       <!-- INDEX -->
       <joint name="${prefix}finger_r_joint5" type="revolute">
-         <parent link="${prefix}rh_5_right_base" />
+         <parent link="${prefix}hx5_d20_right_base" />
          <child link="${prefix}finger_r_link5" />
          <origin xyz="-0.0015 0.03608 0.09575" rpy="0 0 0" />
@@ -205,14 +205,14 @@
             <origin xyz="0 0 0" rpy="0 0 0" />
             <geometry>
-               <mesh filename="${meshes_file_direction}/rh_5_finger_mcp.stl" scale="0.001 0.001 0.001" />
-            </geometry>
-            <material name="grey">
-               <color rgba="0.2 0.2 0.2 1" />
-            </material>
-         </visual>
-         <collision>
-            <origin xyz="0 0 0" rpy="0 0 0" />
-            <geometry>
-               <mesh filename="${meshes_file_direction}/rh_5_finger_mcp.stl" scale="0.001 0.001 0.001" />
+               <mesh filename="${meshes_file_direction}/hx5_d20_finger_mcp.stl" scale="0.001 0.001 0.001" />
+            </geometry>
+            <material name="grey">
+               <color rgba="0.2 0.2 0.2 1" />
+            </material>
+         </visual>
+         <collision>
+            <origin xyz="0 0 0" rpy="0 0 0" />
+            <geometry>
+               <mesh filename="${meshes_file_direction}/hx5_d20_finger_mcp.stl" scale="0.001 0.001 0.001" />
             </geometry>
             <material name="grey">
@@ -240,14 +240,14 @@
             <origin xyz="0 0 0" rpy="0 0 0" />
             <geometry>
-               <mesh filename="${meshes_file_direction}/rh_5_finger_pip.stl" scale="0.001 0.001 0.001" />
-            </geometry>
-            <material name="grey">
-               <color rgba="0.2 0.2 0.2 1" />
-            </material>
-         </visual>
-         <collision>
-            <origin xyz="0 0 0" rpy="0 0 0" />
-            <geometry>
-               <mesh filename="${meshes_file_direction}/rh_5_finger_pip.stl" scale="0.001 0.001 0.001" />
+               <mesh filename="${meshes_file_direction}/hx5_d20_finger_pip.stl" scale="0.001 0.001 0.001" />
+            </geometry>
+            <material name="grey">
+               <color rgba="0.2 0.2 0.2 1" />
+            </material>
+         </visual>
+         <collision>
+            <origin xyz="0 0 0" rpy="0 0 0" />
+            <geometry>
+               <mesh filename="${meshes_file_direction}/hx5_d20_finger_pip.stl" scale="0.001 0.001 0.001" />
             </geometry>
             <material name="grey">
@@ -275,14 +275,14 @@
             <origin xyz="0 0 0" rpy="0 0 0" />
             <geometry>
-               <mesh filename="${meshes_file_direction}/rh_5_finger_dip.stl" scale="0.001 0.001 0.001" />
-            </geometry>
-            <material name="grey">
-               <color rgba="0.2 0.2 0.2 1" />
-            </material>
-         </visual>
-         <collision>
-            <origin xyz="0 0 0" rpy="0 0 0" />
-            <geometry>
-               <mesh filename="${meshes_file_direction}/rh_5_finger_dip.stl" scale="0.001 0.001 0.001" />
+               <mesh filename="${meshes_file_direction}/hx5_d20_finger_dip.stl" scale="0.001 0.001 0.001" />
+            </geometry>
+            <material name="grey">
+               <color rgba="0.2 0.2 0.2 1" />
+            </material>
+         </visual>
+         <collision>
+            <origin xyz="0 0 0" rpy="0 0 0" />
+            <geometry>
+               <mesh filename="${meshes_file_direction}/hx5_d20_finger_dip.stl" scale="0.001 0.001 0.001" />
             </geometry>
             <material name="grey">
@@ -310,14 +310,14 @@
             <origin xyz="0 0 0" rpy="0 0 0" />
             <geometry>
-               <mesh filename="${meshes_file_direction}/rh_5_finger_tip.stl" scale="0.001 0.001 0.001" />
-            </geometry>
-            <material name="grey">
-               <color rgba="0.2 0.2 0.2 1" />
-            </material>
-         </visual>
-         <collision>
-            <origin xyz="0 0 0" rpy="0 0 0" />
-            <geometry>
-               <mesh filename="${meshes_file_direction}/rh_5_finger_tip.stl" scale="0.001 0.001 0.001" />
+               <mesh filename="${meshes_file_direction}/hx5_d20_finger_tip.stl" scale="0.001 0.001 0.001" />
+            </geometry>
+            <material name="grey">
+               <color rgba="0.2 0.2 0.2 1" />
+            </material>
+         </visual>
+         <collision>
+            <origin xyz="0 0 0" rpy="0 0 0" />
+            <geometry>
+               <mesh filename="${meshes_file_direction}/hx5_d20_finger_tip.stl" scale="0.001 0.001 0.001" />
             </geometry>
             <material name="grey">
@@ -351,5 +351,5 @@
       <!-- MIDDLE -->
       <joint name="${prefix}finger_r_joint9" type="revolute">
-         <parent link="${prefix}rh_5_right_base" />
+         <parent link="${prefix}hx5_d20_right_base" />
          <child link="${prefix}finger_r_link9" />
          <origin xyz="-0.0015 0.00908 0.10353" rpy="0 0 0" />
@@ -362,14 +362,14 @@
             <origin xyz="0 0 0" rpy="0 0 0" />
             <geometry>
-               <mesh filename="${meshes_file_direction}/rh_5_finger_mcp.stl" scale="0.001 0.001 0.001" />
-            </geometry>
-            <material name="grey">
-               <color rgba="0.2 0.2 0.2 1" />
-            </material>
-         </visual>
-         <collision>
-            <origin xyz="0 0 0" rpy="0 0 0" />
-            <geometry>
-               <mesh filename="${meshes_file_direction}/rh_5_finger_mcp.stl" scale="0.001 0.001 0.001" />
+               <mesh filename="${meshes_file_direction}/hx5_d20_finger_mcp.stl" scale="0.001 0.001 0.001" />
+            </geometry>
+            <material name="grey">
+               <color rgba="0.2 0.2 0.2 1" />
+            </material>
+         </visual>
+         <collision>
+            <origin xyz="0 0 0" rpy="0 0 0" />
+            <geometry>
+               <mesh filename="${meshes_file_direction}/hx5_d20_finger_mcp.stl" scale="0.001 0.001 0.001" />
             </geometry>
             <material name="grey">
@@ -397,14 +397,14 @@
             <origin xyz="0 0 0" rpy="0 0 0" />
             <geometry>
-               <mesh filename="${meshes_file_direction}/rh_5_finger_pip.stl" scale="0.001 0.001 0.001" />
-            </geometry>
-            <material name="grey">
-               <color rgba="0.2 0.2 0.2 1" />
-            </material>
-         </visual>
-         <collision>
-            <origin xyz="0 0 0" rpy="0 0 0" />
-            <geometry>
-               <mesh filename="${meshes_file_direction}/rh_5_finger_pip.stl" scale="0.001 0.001 0.001" />
+               <mesh filename="${meshes_file_direction}/hx5_d20_finger_pip.stl" scale="0.001 0.001 0.001" />
+            </geometry>
+            <material name="grey">
+               <color rgba="0.2 0.2 0.2 1" />
+            </material>
+         </visual>
+         <collision>
+            <origin xyz="0 0 0" rpy="0 0 0" />
+            <geometry>
+               <mesh filename="${meshes_file_direction}/hx5_d20_finger_pip.stl" scale="0.001 0.001 0.001" />
             </geometry>
             <material name="grey">
@@ -432,14 +432,14 @@
             <origin xyz="0 0 0" rpy="0 0 0" />
             <geometry>
-               <mesh filename="${meshes_file_direction}/rh_5_finger_dip.stl" scale="0.001 0.001 0.001" />
-            </geometry>
-            <material name="grey">
-               <color rgba="0.2 0.2 0.2 1" />
-            </material>
-         </visual>
-         <collision>
-            <origin xyz="0 0 0" rpy="0 0 0" />
-            <geometry>
-               <mesh filename="${meshes_file_direction}/rh_5_finger_dip.stl" scale="0.001 0.001 0.001" />
+               <mesh filename="${meshes_file_direction}/hx5_d20_finger_dip.stl" scale="0.001 0.001 0.001" />
+            </geometry>
+            <material name="grey">
+               <color rgba="0.2 0.2 0.2 1" />
+            </material>
+         </visual>
+         <collision>
+            <origin xyz="0 0 0" rpy="0 0 0" />
+            <geometry>
+               <mesh filename="${meshes_file_direction}/hx5_d20_finger_dip.stl" scale="0.001 0.001 0.001" />
             </geometry>
             <material name="grey">
@@ -467,14 +467,14 @@
             <origin xyz="0 0 0" rpy="0 0 0" />
             <geometry>
-               <mesh filename="${meshes_file_direction}/rh_5_finger_tip.stl" scale="0.001 0.001 0.001" />
-            </geometry>
-            <material name="grey">
-               <color rgba="0.2 0.2 0.2 1" />
-            </material>
-         </visual>
-         <collision>
-            <origin xyz="0 0 0" rpy="0 0 0" />
-            <geometry>
-               <mesh filename="${meshes_file_direction}/rh_5_finger_tip.stl" scale="0.001 0.001 0.001" />
+               <mesh filename="${meshes_file_direction}/hx5_d20_finger_tip.stl" scale="0.001 0.001 0.001" />
+            </geometry>
+            <material name="grey">
+               <color rgba="0.2 0.2 0.2 1" />
+            </material>
+         </visual>
+         <collision>
+            <origin xyz="0 0 0" rpy="0 0 0" />
+            <geometry>
+               <mesh filename="${meshes_file_direction}/hx5_d20_finger_tip.stl" scale="0.001 0.001 0.001" />
             </geometry>
             <material name="grey">
@@ -508,5 +508,5 @@
       <!-- RING -->
       <joint name="${prefix}finger_r_joint13" type="revolute">
-         <parent link="${prefix}rh_5_right_base" />
+         <parent link="${prefix}hx5_d20_right_base" />
          <child link="${prefix}finger_r_link13" />
          <origin xyz="-0.0015 -0.01792 0.09775" rpy="0 0 0" />
@@ -519,14 +519,14 @@
             <origin xyz="0 0 0" rpy="0 0 0" />
             <geometry>
-               <mesh filename="${meshes_file_direction}/rh_5_finger_mcp.stl" scale="0.001 0.001 0.001" />
-            </geometry>
-            <material name="grey">
-               <color rgba="0.2 0.2 0.2 1" />
-            </material>
-         </visual>
-         <collision>
-            <origin xyz="0 0 0" rpy="0 0 0" />
-            <geometry>
-               <mesh filename="${meshes_file_direction}/rh_5_finger_mcp.stl" scale="0.001 0.001 0.001" />
+               <mesh filename="${meshes_file_direction}/hx5_d20_finger_mcp.stl" scale="0.001 0.001 0.001" />
+            </geometry>
+            <material name="grey">
+               <color rgba="0.2 0.2 0.2 1" />
+            </material>
+         </visual>
+         <collision>
+            <origin xyz="0 0 0" rpy="0 0 0" />
+            <geometry>
+               <mesh filename="${meshes_file_direction}/hx5_d20_finger_mcp.stl" scale="0.001 0.001 0.001" />
             </geometry>
             <material name="grey">
@@ -554,14 +554,14 @@
             <origin xyz="0 0 0" rpy="0 0 0" />
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
File: ffw_description/urdf/ffw_bh5_rev1_follower/ffw_bh5_follower.urdf.xacro (robot description, xacro)
@@ -9,6 +9,6 @@
   <xacro:include filename="$(find ffw_description)/urdf/common/follower/ffw_follower_body.xacro" />
   <!-- <xacro:include filename="$(find ffw_description)/urdf/common/rh_p12_rn_a/rh_p12_rn_a.urdf.xacro" /> -->
-  <xacro:include filename="$(find ffw_description)/urdf/common/rh_5_left/rh_5_left.urdf.xacro" />
-  <xacro:include filename="$(find ffw_description)/urdf/common/rh_5_right/rh_5_right.urdf.xacro" />
+  <xacro:include filename="$(find ffw_description)/urdf/common/hx5_d20_left/hx5_d20_left.urdf.xacro" />
+  <xacro:include filename="$(find ffw_description)/urdf/common/hx5_d20_right/hx5_d20_right.urdf.xacro" />
   <xacro:include filename="$(find ffw_description)/ros2_control/$(arg model)/ffw_bh5_follower.ros2_control.xacro" />
   <xacro:include filename="$(find ffw_description)/ros2_control/$(arg model)/ffw_bh5_follower_left.ros2_control.xacro" />
@@ -47,13 +47,13 @@
     <origin xyz="0.0055 0 1.4316" rpy="0 0 0" />
   </xacro:ffw_follower_body>
-  <xacro:rh_5_left parent="$(arg prefix)arm_l_link7" prefix="$(arg prefix)">
+  <xacro:hx5_d20_left parent="$(arg prefix)arm_l_link7" prefix="$(arg prefix)">
     <origin xyz="0 0 -0.078" rpy="0 3.14159265359 1.5708"/>
-  </xacro:rh_5_left>
+  </xacro:hx5_d20_left>
   <!-- <xacro:rh_p12_rn_a parent="$(arg prefix)arm_l_link7" prefix="$(arg prefix)gripper_l_">
     <origin xyz="0 0 -0.078" rpy="0 3.14159265359 3.14159265359"/>
   </xacro:rh_p12_rn_a> -->
-  <xacro:rh_5_right parent="$(arg prefix)arm_r_link7" prefix="$(arg prefix)">
+  <xacro:hx5_d20_right parent="$(arg prefix)arm_r_link7" prefix="$(arg prefix)">
     <origin xyz="0 0 -0.078" rpy="0 3.14159265359 -1.5708"/>
-  </xacro:rh_5_right>
+  </xacro:hx5_d20_right>
   <xacro:ffw_bh5_follower_system
     use_sim="$(arg use_sim)"
