Commit message: Modified for finger tip sensor
Signed-off-by: Wonho Yun <ywh@robotis.com>

File: ffw_description/ros2_control/ffw_bh5_rev1_follower/ffw_bh5_follower_one.ros2_control.xacro (robot description, xacro)
@@ -533,25 +533,25 @@
         <param name="SyncTable 1 ID 3">113</param>
         <param name="SyncTable 1 ID 4">114</param>
-        <param name="SyncTable 1 ID 5">255</param>
+        <param name="SyncTable 1 ID 5">115</param>
         <param name="SyncTable 2 ID 1">121</param>
         <param name="SyncTable 2 ID 2">122</param>
         <param name="SyncTable 2 ID 3">123</param>
         <param name="SyncTable 2 ID 4">124</param>
-        <param name="SyncTable 2 ID 5">255</param>
+        <param name="SyncTable 2 ID 5">125</param>
         <param name="SyncTable 3 ID 1">131</param>
         <param name="SyncTable 3 ID 2">132</param>
         <param name="SyncTable 3 ID 3">133</param>
         <param name="SyncTable 3 ID 4">134</param>
-        <param name="SyncTable 3 ID 5">255</param>
+        <param name="SyncTable 3 ID 5">135</param>
         <param name="SyncTable 4 ID 1">116</param>
         <param name="SyncTable 4 ID 2">117</param>
         <param name="SyncTable 4 ID 3">118</param>
         <param name="SyncTable 4 ID 4">119</param>
-        <param name="SyncTable 4 ID 5">255</param>
+        <param name="SyncTable 4 ID 5">120</param>
         <param name="SyncTable 5 ID 1">126</param>
         <param name="SyncTable 5 ID 2">127</param>
         <param name="SyncTable 5 ID 3">128</param>
         <param name="SyncTable 5 ID 4">129</param>
-        <param name="SyncTable 5 ID 5">255</param>
+        <param name="SyncTable 5 ID 5">130</param>
         <param name="SyncTable 1 Read Address 1">224</param>
         <param name="SyncTable 1 Read Address 2">224</param>
@@ -563,5 +563,5 @@
         <param name="SyncTable 1 Read Size 3">6</param>
         <param name="SyncTable 1 Read Size 4">6</param>
-        <param name="SyncTable 1 Read Size 5">0</param>
+        <param name="SyncTable 1 Read Size 5">9</param>
         <param name="SyncTable 1 Write Address 1">230</param>
         <param name="SyncTable 1 Write Address 2">230</param>
@@ -583,5 +583,5 @@
         <param name="SyncTable 2 Read Size 3">6</param>
         <param name="SyncTable 2 Read Size 4">6</param>
-        <param name="SyncTable 2 Read Size 5">0</param>
+        <param name="SyncTable 2 Read Size 5">9</param>
         <param name="SyncTable 2 Write Address 1">230</param>
         <param name="SyncTable 2 Write Address 2">230</param>
@@ -603,5 +603,5 @@
         <param name="SyncTable 3 Read Size 3">6</param>
         <param name="SyncTable 3 Read Size 4">6</param>
-        <param name="SyncTable 3 Read Size 5">0</param>
+        <param name="SyncTable 3 Read Size 5">9</param>
         <param name="SyncTable 3 Write Address 1">230</param>
         <param name="SyncTable 3 Write Address 2">230</param>
@@ -623,5 +623,5 @@
         <param name="SyncTable 4 Read Size 3">6</param>
         <param name="SyncTable 4 Read Size 4">6</param>
-        <param name="SyncTable 4 Read Size 5">0</param>
+        <param name="SyncTable 4 Read Size 5">9</param>
         <param name="SyncTable 4 Write Address 1">230</param>
         <param name="SyncTable 4 Write Address 2">230</param>
@@ -643,5 +643,5 @@
         <param name="SyncTable 5 Read Size 3">6</param>
         <param name="SyncTable 5 Read Size 4">6</param>
-        <param name="SyncTable 5 Read Size 5">0</param>
+        <param name="SyncTable 5 Read Size 5">9</param>
         <param name="SyncTable 5 Write Address 1">230</param>
         <param name="SyncTable 5 Write Address 2">230</param>
@@ -1527,25 +1527,25 @@
         <param name="SyncTable 1 ID 3">163</param>
         <param name="SyncTable 1 ID 4">164</param>
-        <param name="SyncTable 1 ID 5">255</param>
+        <param name="SyncTable 1 ID 5">165</param>
         <param name="SyncTable 2 ID 1">151</param>
         <param name="SyncTable 2 ID 2">152</param>
         <param name="SyncTable 2 ID 3">153</param>
         <param name="SyncTable 2 ID 4">154</param>
-        <param name="SyncTable 2 ID 5">255</param>
+        <param name="SyncTable 2 ID 5">155</param>
         <param name="SyncTable 3 ID 1">141</param>
         <param name="SyncTable 3 ID 2">142</param>
         <param name="SyncTable 3 ID 3">143</param>
         <param name="SyncTable 3 ID 4">144</param>
-        <param name="SyncTable 3 ID 5">255</param>
+        <param name="SyncTable 3 ID 5">145</param>
         <param name="SyncTable 4 ID 1">156</param>
         <param name="SyncTable 4 ID 2">157</param>
         <param name="SyncTable 4 ID 3">158</param>
         <param name="SyncTable 4 ID 4">159</param>
-        <param name="SyncTable 4 ID 5">255</param>
+        <param name="SyncTable 4 ID 5">160</param>
         <param name="SyncTable 5 ID 1">146</param>
         <param name="SyncTable 5 ID 2">147</param>
         <param name="SyncTable 5 ID 3">148</param>
         <param name="SyncTable 5 ID 4">149</param>
-        <param name="SyncTable 5 ID 5">255</param>
+        <param name="SyncTable 5 ID 5">150</param>
         <param name="SyncTable 1 Read Address 1">224</param>
         <param name="SyncTable 1 Read Address 2">224</param>
@@ -1557,5 +1557,5 @@
         <param name="SyncTable 1 Read Size 3">6</param>
         <param name="SyncTable 1 Read Size 4">6</param>
-        <param name="SyncTable 1 Read Size 5">0</param>
+        <param name="SyncTable 1 Read Size 5">9</param>
         <param name="SyncTable 1 Write Address 1">230</param>
         <param name="SyncTable 1 Write Address 2">230</param>
@@ -1577,5 +1577,5 @@
         <param name="SyncTable 2 Read Size 3">6</param>
         <param name="SyncTable 2 Read Size 4">6</param>
-        <param name="SyncTable 2 Read Size 5">0</param>
+        <param name="SyncTable 2 Read Size 5">9</param>
         <param name="SyncTable 2 Write Address 1">230</param>
         <param name="SyncTable 2 Write Address 2">230</param>
@@ -1597,5 +1597,5 @@
         <param name="SyncTable 3 Read Size 3">6</param>
         <param name="SyncTable 3 Read Size 4">6</param>
-        <param name="SyncTable 3 Read Size 5">0</param>
+        <param name="SyncTable 3 Read Size 5">9</param>
         <param name="SyncTable 3 Write Address 1">230</param>
         <param name="SyncTable 3 Write Address 2">230</param>
@@ -1617,5 +1617,5 @@
         <param name="SyncTable 4 Read Size 3">6</param>
         <param name="SyncTable 4 Read Size 4">6</param>
-        <param name="SyncTable 4 Read Size 5">0</param>
+        <param name="SyncTable 4 Read Size 5">9</param>
         <param name="SyncTable 4 Write Address 1">230</param>
         <param name="SyncTable 4 Write Address 2">230</param>
@@ -1637,5 +1637,5 @@
         <param name="SyncTable 5 Read Size 3">6</param>
         <param name="SyncTable 5 Read Size 4">6</param>
-        <param name="SyncTable 5 Read Size 5">0</param>
+        <param name="SyncTable 5 Read Size 5">9</param>
         <param name="SyncTable 5 Write Address 1">230</param>
         <param name="SyncTable 5 Write Address 2">230</param>

File: ffw_description/urdf/ffw_bh5_rev1_follower/ffw_bh5_follower.urdf.xacro (robot description, xacro)
@@ -8,10 +8,7 @@
   <xacro:arg name="model" default="ffw_bh5_rev1_follower" />
   <xacro:include filename="$(find ffw_description)/urdf/common/follower/ffw_follower_body.xacro" />
-  <!-- <xacro:include filename="$(find ffw_description)/urdf/common/rh_p12_rn_a/rh_p12_rn_a.urdf.xacro" /> -->
   <xacro:include filename="$(find ffw_description)/urdf/common/hx5_d20_left/hx5_d20_left.urdf.xacro" />
   <xacro:include filename="$(find ffw_description)/urdf/common/hx5_d20_right/hx5_d20_right.urdf.xacro" />
-  <xacro:include filename="$(find ffw_description)/ros2_control/$(arg model)/ffw_bh5_follower_one.ros2_control.xacro" />
-<!--
-  <xacro:include filename="$(find ffw_description)/ros2_control/$(arg model)/ffw_bh5_follower_left.ros2_control.xacro" /> -->
+  <xacro:include filename="$(find ffw_description)/ros2_control/$(arg model)/ffw_bh5_follower.ros2_control.xacro" />
   <xacro:include filename="$(find ffw_description)/gazebo/ffw_bh5_rev1_follower/ffw_bh5_follower.gazebo.xacro" />
   <link name="world"/>
@@ -51,7 +48,4 @@
     <origin xyz="0 0 -0.078" rpy="0 3.14159265359 1.5708"/>
   </xacro:hx5_d20_left>
-  <!-- <xacro:rh_p12_rn_a parent="$(arg prefix)arm_l_link7" prefix="$(arg prefix)gripper_l_">
-    <origin xyz="0 0 -0.078" rpy="0 3.14159265359 3.14159265359"/>
-  </xacro:rh_p12_rn_a> -->
   <xacro:hx5_d20_right parent="$(arg prefix)arm_r_link7" prefix="$(arg prefix)">
     <origin xyz="0 0 -0.078" rpy="0 3.14159265359 -1.5708"/>
@@ -61,8 +55,4 @@
     use_fake_hardware="$(arg use_fake_hardware)"
     fake_sensor_commands="$(arg fake_sensor_commands)"/>
-  <!-- <xacro:ffw_bh5_follower_left_system
-    use_sim="$(arg use_sim)"
-    use_fake_hardware="$(arg use_fake_hardware)"
-    fake_sensor_commands="$(arg fake_sensor_commands)"/> -->
   <gazebo>
       <plugin filename="gz_ros2_control-system" name="gz_ros2_control::GazeboSimROS2ControlPlugin">
