Commit message: feat: Add left and right Lidar joints and links to the URDF

File: ffw_description/urdf/ffw_sg2_rev1_follower/ffw_sg2_follower.urdf.xacro (robot description, xacro)
@@ -36,4 +36,20 @@
        izz="2.846139500e+04" />
     </inertial>
+  </link>
+  <!-- Left Lidar -->
+  <joint name="$(arg prefix)lidar_l_joint" type="fixed">
+    <parent link="$(arg prefix)base_link"/>
+    <child link="$(arg prefix)lidar_l_link"/>
+    <origin xyz="-0.111881 0.240 0.34432" rpy="0 0 0"/>
+  </joint>
+  <link name="$(arg prefix)lidar_l_link">
+  </link>
+  <!-- Right Lidar -->
+  <joint name="$(arg prefix)lidar_r_joint" type="fixed">
+    <parent link="$(arg prefix)base_link"/>
+    <child link="$(arg prefix)lidar_r_link"/>
+    <origin xyz="-0.111881 -0.240 0.34432" rpy="0 0 0"/>
+  </joint>
+  <link name="$(arg prefix)lidar_r_link">
   </link>
   <link name="$(arg prefix)lift_link">

Commit message: feat: Add world link and fixed joint to base link in URDF
Signed-off-by: Heewon Lee <7dlgmldnjs7@gmail.com>

File: ffw_description/urdf/ffw_sg2_rev1_follower/ffw_sg2_follower.urdf.xacro (robot description, xacro)
@@ -13,4 +13,10 @@
   <xacro:include filename="$(find ffw_description)/ros2_control/$(arg model)/ffw_sg2_sensor.ros2_control.xacro" />
   <xacro:include filename="$(find ffw_description)/gazebo/$(arg model)/ffw_sg2_follower.gazebo.xacro" />
+  <link name="world"/>
+  <joint name="$(arg prefix)world_fixed" type="fixed">
+    <parent link="world"/>
+    <child link="$(arg prefix)base_link"/>
+    <origin xyz="0.0 0.0 0.0" rpy="0 0 0"/>
+  </joint>
   <link name="$(arg prefix)base_link">
     <visual>

Commit message: refactor: Remove unused world link and joint from URDF file
Signed-off-by: Heewon Lee <7dlgmldnjs7@gmail.com>

File: ffw_description/urdf/ffw_sg2_rev1_follower/ffw_sg2_follower.urdf.xacro (robot description, xacro)
@@ -13,10 +13,4 @@
   <xacro:include filename="$(find ffw_description)/ros2_control/$(arg model)/ffw_sg2_sensor.ros2_control.xacro" />
   <xacro:include filename="$(find ffw_description)/gazebo/$(arg model)/ffw_sg2_follower.gazebo.xacro" />
-  <link name="world"/>
-  <joint name="$(arg prefix)world_fixed" type="fixed">
-    <parent link="world"/>
-    <child link="$(arg prefix)base_link"/>
-    <origin xyz="0.0 0.0 0.0" rpy="0 0 0"/>
-  </joint>
   <link name="$(arg prefix)base_link">
     <visual>
