Commit message: teleop , moveit and gazebo

File: ffw_description/urdf/common/follower/ffw_follower_body.xacro (robot description, xacro)
@@ -144,5 +144,5 @@
          <origin xyz="0 0.123 0" rpy="0 0 0" />
          <axis xyz="1 0 0" />
-         <limit velocity="4.8" effort="1000" lower="0.0" upper="3.14" />
+         <limit velocity="4.8" effort="1000" lower="-0.1" upper="3.14" />
          <dynamics damping="0.1" />
       </joint>
@@ -371,5 +371,5 @@
          <origin xyz="0 -0.123 0" rpy="0 0 0" />
          <axis xyz="1 0 0" />
-         <limit velocity="4.8" effort="1000" lower="-3.14" upper="0" />
+         <limit velocity="4.8" effort="1000" lower="-3.14" upper="0.1" />
          <dynamics damping="0.1" />
       </joint>

File: ffw_description/urdf/ffw_sg2_rev1_follower/ffw_sg2_follower.urdf (robot description, URDF)
Before this commit: robot ffw_sg2_follower, 40 links, 39 joints
Joints:
- joint arm_l_joint2: limit lower=0.0 upper=3.14 effort=1000 velocity=4.8 -> lower=-0.1 upper=3.14 effort=1000 velocity=4.8
- joint arm_r_joint2: limit lower=-3.14 upper=0 effort=1000 velocity=4.8 -> lower=-3.14 upper=0.1 effort=1000 velocity=4.8
