Commit message: ffw_description, ffw_bringup: bake the OAK-D nominal mount offset into the URDF as camera_calibration_link
Previously the whole zedm_left_camera_optical_frame -> head_camera_frame
transform (ZED-to-OAK-D nominal offset AND identity rotation) lived
entirely in the oakd_cam_static_tf static_transform_publisher's
arguments in the *_follower_ai_stream launch files, invisible to the
robot model itself.

Split it in two:
  - camera_calibration_link (new, in ffw_follower_body.xacro): a real
    URDF link carrying the ORIGINAL nominal mount offset (+31.5mm x,
    identity rotation -- ZED-to-OAK-D center shift), child of
    zedm_left_camera_optical_frame.
  - oakd_cam_static_tf (updated, in both stream launch files): now goes
    camera_calibration_link -> head_camera_frame, carrying only the
    small residual correction solved from the AprilTag-board head-sweep
    calibration (translation ~0.6-1.6cm, rotation ~1 deg, condition
    number ~10, residual RMS ~0.2cm after outlier removal -- see
    ffw_depthai/scripts/sweep_and_solve_camera_calibration.py and
    camera_calib_lib.py).

head_camera_frame itself is unchanged as a runtime
static_transform_publisher child (still not a URDF link, so it's not
double-parented against /head_camera_tf's own resolution), and its
absolute pose relative to head_link2 is unchanged to within the small
solved correction -- this just makes the correction an explicit, named,
independently-tunable offset instead of a number folded into the
mount's own arguments.

Co-Authored-By: Claude Sonnet 5 <noreply@anthropic.com>
Claude-Session: https://claude.ai/code/session_01FoS1C59Fqfe76y6AS1FYbi

File: ffw_description/urdf/common/follower/ffw_follower_body.xacro (robot description, xacro)
@@ -107,4 +107,19 @@
          <origin xyz="0.0238122 -0.00651797 -0.0242094" rpy="0 0 0" />
       </joint>
+      <!-- The OAK-D replacing the ZED in the same physical mount bracket:
+           this is the ORIGINAL, uncorrected mount offset (what the
+           head_camera_frame static_transform_publisher used before it was
+           calibrated). head_camera_frame itself stays a runtime
+           static_transform_publisher child of camera_calibration_link (see
+           ffw_bringup's *_follower_ai_stream launch files) rather than a
+           URDF link, so it is not double parented, but the small measured
+           correction now lives there as an explicit, named offset instead of
+           being folded invisibly into that node's arguments. -->
+      <link name="camera_calibration_link" />
+      <joint name="camera_calibration_joint" type="fixed">
+         <parent link="zedm_left_camera_optical_frame"/>
+         <child link="camera_calibration_link"/>
+         <origin xyz="0.0315 0 0" rpy="0 0 0" />
+      </joint>
       <joint name="${prefix}arm_l_joint1" type="revolute">
          <parent link="${prefix}arm_base_link" />
