Commit message: robot-update: ffw_bringup/XACRO_BLOCK_PARAM_BUG.md ffw_bringup/XM430_GRIPPER_SETUP.md ffw_bringup/config/ffw_sg2_s...

File: ffw_description/urdf/common/rh_p12_rn_a/rh_p12_rn_a.urdf.xacro (robot description, xacro)
@@ -2,10 +2,10 @@
 <!-- rh_p12_rn_a gripper -->
 <robot xmlns:xacro="http://www.ros.org/wiki/xacro">
-  <xacro:macro name="rh_p12_rn_a" params="prefix parent *origin">
+  <xacro:macro name="rh_p12_rn_a" params="prefix parent origin_xyz origin_rpy">
     <xacro:property
       name="meshes_file_direction"
       value="package://ffw_description/meshes/common/rh_p12_rn_a"/>
     <joint name="${prefix}joint" type="fixed">
-      <xacro:insert_block name="origin" />
+      <origin xyz="${origin_xyz}" rpy="${origin_rpy}"/>
       <parent link="${parent}"/>
       <child link="${prefix}rh_p12_rn_base" />

File: ffw_description/urdf/ffw_bg2_rev2_follower/ffw_bg2_follower.urdf.xacro (robot description, xacro)
@@ -42,10 +42,8 @@
     <origin xyz="0.053 0 1.2846" rpy="0 0 0" />
   </xacro:ffw_follower_body>
-  <xacro:rh_p12_rn_a parent="$(arg prefix)arm_l_link7" prefix="$(arg prefix)gripper_l_">
-    <origin xyz="0 0 -0.05" rpy="0 3.14159265359 3.14159265359"/>
-  </xacro:rh_p12_rn_a>
-  <xacro:rh_p12_rn_a parent="$(arg prefix)arm_r_link7" prefix="$(arg prefix)gripper_r_">
-    <origin xyz="0 0 -0.05" rpy="0 3.14159265359 3.14159265359"/>
-  </xacro:rh_p12_rn_a>
+  <xacro:rh_p12_rn_a parent="$(arg prefix)arm_l_link7" prefix="$(arg prefix)gripper_l_"
+    origin_xyz="0 0 -0.05" origin_rpy="0 3.14159265359 3.14159265359"/>
+  <xacro:rh_p12_rn_a parent="$(arg prefix)arm_r_link7" prefix="$(arg prefix)gripper_r_"
+    origin_xyz="0 0 -0.05" origin_rpy="0 3.14159265359 3.14159265359"/>
   <xacro:ffw_bg2_follower_system
     use_sim="$(arg use_sim)"

File: ffw_description/urdf/ffw_bg2_rev3_follower/ffw_bg2_follower.urdf.xacro (robot description, xacro)
@@ -42,10 +42,8 @@
     <origin xyz="0.053 0 1.2846" rpy="0 0 0" />
   </xacro:ffw_follower_body>
-  <xacro:rh_p12_rn_a parent="$(arg prefix)arm_l_link7" prefix="$(arg prefix)gripper_l_">
-    <origin xyz="0 0 -0.05" rpy="0 3.14159265359 3.14159265359"/>
-  </xacro:rh_p12_rn_a>
-  <xacro:rh_p12_rn_a parent="$(arg prefix)arm_r_link7" prefix="$(arg prefix)gripper_r_">
-    <origin xyz="0 0 -0.05" rpy="0 3.14159265359 3.14159265359"/>
-  </xacro:rh_p12_rn_a>
+  <xacro:rh_p12_rn_a parent="$(arg prefix)arm_l_link7" prefix="$(arg prefix)gripper_l_"
+    origin_xyz="0 0 -0.05" origin_rpy="0 3.14159265359 3.14159265359"/>
+  <xacro:rh_p12_rn_a parent="$(arg prefix)arm_r_link7" prefix="$(arg prefix)gripper_r_"
+    origin_xyz="0 0 -0.05" origin_rpy="0 3.14159265359 3.14159265359"/>
   <xacro:ffw_bg2_follower_system
     use_sim="$(arg use_sim)"

File: ffw_description/urdf/ffw_bg2_rev4_follower/ffw_bg2_follower.urdf.xacro (robot description, xacro)
@@ -45,7 +45,6 @@
     <origin xyz="0.0055 0 1.4316" rpy="0 0 0" />
   </xacro:ffw_follower_body>
-  <xacro:rh_p12_rn_a parent="$(arg prefix)arm_l_link7" prefix="$(arg prefix)gripper_l_">
-    <origin xyz="0 0 -0.078" rpy="0 3.14159265359 3.14159265359"/>
-  </xacro:rh_p12_rn_a>
+  <xacro:rh_p12_rn_a parent="$(arg prefix)arm_l_link7" prefix="$(arg prefix)gripper_l_"
+    origin_xyz="0 0 -0.078" origin_rpy="0 3.14159265359 3.14159265359"/>
   <joint name="$(arg prefix)end_effector_l_joint" type="fixed">
     <parent link="$(arg prefix)arm_l_link7"/>
@@ -64,7 +63,6 @@
     </visual>
   </link>
-  <xacro:rh_p12_rn_a parent="$(arg prefix)arm_r_link7" prefix="$(arg prefix)gripper_r_">
-    <origin xyz="0 0 -0.078" rpy="0 3.14159265359 3.14159265359"/>
-  </xacro:rh_p12_rn_a>
+  <xacro:rh_p12_rn_a parent="$(arg prefix)arm_r_link7" prefix="$(arg prefix)gripper_r_"
+    origin_xyz="0 0 -0.078" origin_rpy="0 3.14159265359 3.14159265359"/>
   <joint name="$(arg prefix)end_effector_r_joint" type="fixed">
     <parent link="$(arg prefix)arm_r_link7"/>

File: ffw_description/urdf/ffw_sg2_smtm/ffw_sg2_smtm.urdf.xacro (robot description, xacro)
@@ -1,17 +1,18 @@
 <?xml version="1.0"?>
-<robot xmlns:xacro="http://www.ros.org/wiki/xacro" name="ffw_sg2_follower">
-  <xacro:property name="meshes_file_direction" value="package://ffw_description/meshes/$(arg model)" />
+<robot xmlns:xacro="http://www.ros.org/wiki/xacro" name="ffw_sg2_smtm">
+  <xacro:property name="meshes_file_direction" value="package://ffw_description/meshes/ffw_sg2_rev1_follower" />
   <xacro:arg name="use_sim" default="false" />
   <xacro:arg name="use_mock_hardware" default="false" />
   <xacro:arg name="mock_sensor_commands" default="false" />
   <xacro:arg name="prefix" default="" />
-  <xacro:arg name="model" default="ffw_sg2_rev1_follower" />
-  <xacro:arg name="ros2_control_type" default="ffw_sg2_follower" />
+  <xacro:arg name="model" default="ffw_sg2_smtm" />
+  <xacro:arg name="ros2_control_type" default="ffw_sg2_smtm" />
   <xacro:include filename="$(find ffw_description)/urdf/common/follower/ffw_follower_body.xacro" />
+  <xacro:include filename="$(find ffw_description)/urdf/common/xm430_gripper/xm430_gripper.urdf.xacro" />
   <xacro:include filename="$(find ffw_description)/urdf/common/rh_p12_rn_a/rh_p12_rn_a.urdf.xacro" />
   <xacro:include filename="$(find ffw_description)/ros2_control/$(arg model)/$(arg ros2_control_type).ros2_control.xacro" />
   <xacro:include filename="$(find ffw_description)/ros2_control/$(arg model)/ffw_sg2_base.ros2_control.xacro" />
   <xacro:include filename="$(find ffw_description)/ros2_control/$(arg model)/ffw_sg2_sensor.ros2_control.xacro" />
-  <xacro:include filename="$(find ffw_description)/gazebo/$(arg model)/ffw_sg2_follower.gazebo.xacro" />
+  <xacro:include filename="$(find ffw_description)/gazebo/$(arg model)/ffw_sg2_smtm.gazebo.xacro" />
   <link name="$(arg prefix)base_link">
     <visual>
@@ -60,6 +61,4 @@
     <origin xyz="-0.111881 -0.240 0.34432" rpy="0 0 -1.57079632679"/>
   </joint>
-  <!-- <link name="$(arg prefix)lidar_r_link">
-  </link> -->
   <joint name="$(arg prefix)imu_joint" type="fixed">
     <parent link="$(arg prefix)base_link"/>
@@ -112,8 +111,9 @@
   </joint>
   <!-- Gazebo plugins/sensors -->
-  <xacro:ffw_sg2_follower_gazebo prefix="$(arg prefix)" />
+  <xacro:ffw_sg2_smtm_gazebo prefix="$(arg prefix)" />
   <xacro:ffw_follower_body parent="$(arg prefix)base_link" prefix="$(arg prefix)">
     <origin xyz="-0.0199 0 1.4316" rpy="0 0 0" />
   </xacro:ffw_follower_body>
+  <!-- Left arm - RH-P12-RN-A gripper (unchanged from original follower) -->
   <xacro:rh_p12_rn_a parent="$(arg prefix)arm_l_link7" prefix="$(arg prefix)gripper_l_"
     origin_xyz="0 0 -0.078" origin_rpy="0 3.14159265359 3.14159265359"/>
@@ -134,6 +134,7 @@
     </visual>
   </link>
-  <xacro:rh_p12_rn_a parent="$(arg prefix)arm_r_link7" prefix="$(arg prefix)gripper_r_"
-    origin_xyz="0 0 -0.078" origin_rpy="0 3.14159265359 3.14159265359"/>
+  <!-- Right arm - XM430 gripper -->
+  <xacro:xm430_gripper parent="$(arg prefix)arm_r_link7" prefix="$(arg prefix)gripper_r_"
+    origin_xyz="0 0 -0.11" origin_rpy="0 1.57079632679 0"/>
   <joint name="$(arg prefix)end_effector_r_joint" type="fixed">
     <parent link="$(arg prefix)arm_r_link7"/>
@@ -200,10 +201,4 @@
       </material>
     </visual>
-    <!-- <collision>
-      <origin xyz="0 0 0" rpy="0 0 0" />
-      <geometry>
-        <mesh filename="${meshes_file_direction}/left_wheel_drive_link.stl" scale="0.001 0.001 0.001" />
-      </geometry>
-    </collision> -->
     <collision>
       <origin xyz="0 0 0" rpy="1.5708 0 0"/>
@@ -268,10 +263,4 @@
       </material>
     </visual>
-    <!-- <collision>
-      <origin xyz="0 0 0" rpy="0 0 0" />
-      <geometry>
-        <mesh filename="${meshes_file_direction}/right_wheel_drive_link.stl" scale="0.001 0.001 0.001" />
-      </geometry>
-    </collision> -->
     <collision>
       <origin xyz="0 0 0" rpy="1.5708 0 0"/>
@@ -342,10 +331,4 @@
       </geometry>
     </collision>
-    <!-- <collision>
-      <origin xyz="0 0 0" rpy="0 0 0" />
-      <geometry>
-        <mesh filename="${meshes_file_direction}/rear_wheel_drive_link.stl" scale="0.001 0.001 0.001" />
-      </geometry>
-    </collision> -->
     <inertial>
        <origin xyz="0.000000000e+00 1.499601700e-03 0.000000000e+00" />
@@ -356,5 +339,5 @@
     </inertial>
   </link>
-  <xacro:ffw_sg2_follower_system
+  <xacro:ffw_sg2_smtm_system
     use_sim="$(arg use_sim)"
     use_mock_hardware="$(arg use_mock_hardware)"
@@ -370,5 +353,5 @@
   <gazebo>
       <plugin filename="gz_ros2_control-system" name="gz_ros2_control::GazeboSimROS2ControlPlugin">
-        <parameters>$(find ffw_bringup)/config/$(arg model)/ffw_sg2_follower_ai_hardware_controller.yaml</parameters>
+        <parameters>$(find ffw_bringup)/config/$(arg model)/ffw_sg2_smtm_ai_hardware_controller.yaml</parameters>
       </plugin>
   </gazebo>
